File: starbie.kicad_sch (KiCad schematic)
At the start: 8 parts, among them J1 Conn_01x04_Pin, J2 Conn_01x08_Pin, SW1 SW_Push, SW2 SW_Push, SW3 SW_SPST, U1 DHT11, U2 XIAO-ESP32-C3-SMD

Commit message: Made a footprint for a rocker power switch
I couldnt find the footprint online so i had to make it myself
Parts:
- SW3: footprint (none) -> Imported Parts:10.4x15mm rocker switch
Changed lines of the file:
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@@
 			)
 		)
-		(property "Footprint" ""
+		(property "Footprint" "Imported Parts:10.4x15mm rocker switch"
 			(at 110.49 24.13 0)
 			(hide yes)
